Commit message: simulacion_robot

File: description/robot.urdf.xacro (robot description, xacro)
@@ -2,3 +2,4 @@
 <robot xmlns:xacro="http://www.ros.org/wiki/xacro"  name="robot">
     <xacro:include filename="robot_base.xacro"/>
+    <xacro:include filename="gazebo_control.xacro"/>
 </robot>

File: description/robot_base.xacro (robot description, xacro)
@@ -67,4 +67,7 @@
         </xacro:inertial_box>
     </link>
+    <gazebo reference="chassis">
+            <material>Gazebo/White</material>
+    </gazebo>
 <!-- Si se quiere entender con imagen hay una foto de como esta los origenes-->
 <!-- RUEDA IZQUIERDA-->
@@ -101,4 +104,7 @@
     </xacro:inertial_cylinder>
  </link>
+<gazebo reference="left_wheel">
+    <material>Gazebo/Blue</material>
+</gazebo>
 <!-- RUEDA DERECHA-->
 <joint name="right_wheel_joint" type="continuous">
@@ -127,4 +133,7 @@
     </xacro:inertial_cylinder>
 </link>
+<gazebo reference="right_wheel">
+    <material>Gazebo/Blue</material>
+</gazebo>
 <!-- RUEDA LOCA O CASTER WHEEL-->
 <joint name="caster_wheel_joint" type="fixed">
@@ -151,3 +160,8 @@
     </xacro:inertial_sphere>
 </link>
+<gazebo reference="caster_wheel">
+    <material>Gazebo/Black</material>
+    <mu1 value="0.001"/>
+    <mu2 value="0.001"/>
+</gazebo>
 </robot>
